Commit message: Colours to USD. Previous USD didn't work I think, mis-type in terminal cmd

File: USD_files/moved_motor_urdf_joint_limits/moved_motor_urdf.urdf (robot description, URDF)
Before this commit: robot moved_motor_urdf, 17 links, 16 joints
Joints:
- joint LF_HAA: limit (none) -> lower=-1.5707963267948966 upper=1.5707963267948966 effort=1000 velocity=1000; type continuous -> revolute
- joint LF_HFE: limit (none) -> lower=-3.141592 upper=0.0 effort=1000 velocity=1000; type continuous -> revolute
- joint LF_KFE: limit (none) -> lower=0.3490658503988659 upper=2.9670597283903604 effort=1000 velocity=1000; type continuous -> revolute
- joint LH_HAA: limit (none) -> lower=-1.5707963267948966 upper=1.5707963267948966 effort=1000 velocity=1000; type continuous -> revolute
- joint LH_HFE: limit (none) -> lower=-3.141592 upper=0.0 effort=1000 velocity=1000; type continuous -> revolute
- joint LH_KFE: limit (none) -> lower=0.3490658503988659 upper=2.9670597283903604 effort=1000 velocity=1000; type continuous -> revolute
- joint RF_HAA: limit (none) -> lower=-1.5707963267948966 upper=1.5707963267948966 effort=1000 velocity=1000; type continuous -> revolute
- joint RF_HFE: limit (none) -> lower=-3.141592 upper=0.0 effort=1000 velocity=1000; type continuous -> revolute
- joint RF_KFE: limit (none) -> lower=0.3490658503988659 upper=2.9670597283903604 effort=1000 velocity=1000; type continuous -> revolute
- joint RH_HAA: limit (none) -> lower=-1.5707963267948966 upper=1.5707963267948966 effort=1000 velocity=1000; type continuous -> revolute
- joint RH_HFE: limit (none) -> lower=-3.141592 upper=0.0 effort=1000 velocity=1000; type continuous -> revolute
- joint RH_KFE: limit (none) -> lower=0.3490658503988659 upper=2.9670597283903604 effort=1000 velocity=1000; type continuous -> revolute
